Commit message: feat: transfer lidar and GPS from capybara to gerbil
- gerbil.launch.xml gains launch_lidar (LD19 + laser_filters) and
  launch_gps (u-blox) groups, on /dev/gerbil_lidar and /dev/gerbil_gps
- URDF gains laser_frame link + lidar_joint (mount pose is a TODO)
- nav2 and slam use the LIDAR; depthimage_to_laserscan removed
- laser_filter.yaml ported; foxglove whitelist regains GPS topics
- udev rules cover all three devices; docs cover the ldlidar clone,
  device table, and scan verification

Co-Authored-By: Claude Opus 5 <noreply@anthropic.com>
Claude-Session: https://claude.ai/code/session_01XooinpebaTuuvn3FGVN3Cu

File: src/gerbil_description/urdf/mobile_base.xacro (robot description, xacro)
@@ -161,4 +161,25 @@
     </joint>
     <!-- IMU centered on top of chassis not quite right, doesn't really matter, can add meshes later -->
+    <!-- LIDAR LINK (LD19) -->
+    <link name="laser_frame">
+        <visual>
+            <geometry>
+                <cylinder radius="0.035" length="0.045" />
+            </geometry>
+            <origin xyz="0 0 0" rpy="0 0 0" />
+            <material name="black" />
+        </visual>
+        <collision>
+            <geometry>
+                <cylinder radius="0.035" length="0.045" />
+            </geometry>
+            <origin xyz="0 0 0" rpy="0 0 0" />
+        </collision>
+        <inertial>
+            <mass value="0.2" />
+            <origin xyz="0 0 0" rpy="0 0 0" />
+            <inertia ixx="0.0001" ixy="0" ixz="0" iyy="0.0001" iyz="0" izz="0.0001" />
+        </inertial>
+    </link>
     <joint name="imu_joint" type="fixed">
         <parent link="base_link" />
@@ -172,3 +193,12 @@
         <origin xyz="${base_length / 2.0 - 0.02} 0 ${base_height + 0.015}" rpy="0 0 0" />
     </joint>
+    <!-- LIDAR mounted on the chassis top, centred.
+         TODO: measure the real mount position and yaw. The rpy below assumes
+         the same 90 deg clockwise mounting as Capybara; verify in Foxglove
+         that an object in front of the robot appears in front on /scan. -->
+    <joint name="lidar_joint" type="fixed">
+        <parent link="base_link" />
+        <child link="laser_frame" />
+        <origin xyz="0 0 ${base_height + 0.023}" rpy="0 0 -1.5708" />
+    </joint>
 </robot>
